File: Human_Tracker.kicad_pcb (KiCad board)
At the start: 4 copper layers, 200 x 50 mm, 59 parts, among them U1 TPS54233QDRQ1, U2 ICS-43434_C5656610, U3 ICS-43434_C5656610, U4 ADM7172ACPZ-3.3-R7, U5 BME680, U6 ESP32-S3-WROOM-1(N16R8), U7 MLX90640ESF-BAB-000-TU, U8 FRC0805F1400TS 140

Commit message: commit
Parts:
- H2: moved to B.Cu
- moved R9 3.16 mm to (172.3, 66.6)
- moved R10 1.33 mm to (172.4, 68.7)
Connections:
- net Net-(U6-IO19) renamed r_D+
- net Net-(U6-IO20) renamed r_D-
Routing:
- net /D+: track 0.00 -> 29.5 mm, vias 0 -> 2
- net /D-: track 0.00 -> 29.4 mm, vias 0 -> 2
- net GND: track 156.7 -> 176.2 mm, vias 9 -> 14
- net Net-(USB1-CC2): track 0.00 -> 6.35 mm, vias 0 -> 1
- net +3.3V: track 113.3 -> 118.9 mm, vias 9 -> 11
- net /UWB_RST: track 176.8 -> 180.3 mm
- net r_D+: track 35.1 -> 38.3 mm, vias 1 -> 2
- net Net-(U4-EN): track 11.1 -> 14.4 mm
- net Net-(U1-EN): track 4.30 -> 6.50 mm
- net r_D-: track 40.0 -> 38.2 mm
- net /UWB_INT: track 178.6 -> 180.2 mm
- net /UWB_WAKEUP: track 165.7 -> 166.4 mm
- net /SCLK: track 149.8 -> 150.4 mm

Commit message: j'ai changé la paires différentielle et j'ai ajouter les DRC the jldpcb
Parts:
- removed R10, R9: 22, lcsc_footprints:C17414_R0805
- moved C9 28.0 mm to (164.9, 32.5), turned to 90 degrees
- moved C8 27.8 mm to (167.1, 32.5), turned to 90 degrees
Connections:
- H2 pad 13: r_D+ -> /D+
- H2 pad 14: r_D- -> /D-
- U6 pad 13: r_D+ -> /D+
- U6 pad 14: r_D- -> /D-
Routing:
- net r_D+: track 38.3 -> 0.00 mm, vias 2 -> 0
- net r_D-: track 38.2 -> 0.00 mm, vias 2 -> 0
- net /D+: track 29.5 -> 55.5 mm, vias 2 -> 0
- net /D-: track 29.4 -> 54.8 mm, vias 2 -> 0
- net /MISO: track 168.8 -> 160.8 mm
- net /MOSI: track 159.6 -> 154.2 mm
- net /SCLK: track 150.4 -> 146.1 mm, vias 1 -> 3
- net /UWB_INT: track 180.2 -> 176.4 mm, vias 0 -> 2
- net Net-(WIRELM1-GPIO3): track 12.6 -> 14.9 mm
- net /UWB_WAKEUP: track 166.4 -> 164.8 mm, vias 3 -> 5
- net /UWB_RST: track 180.3 -> 179.0 mm
- net Net-(WIRELM1-GPIO2): vias 1 -> 0
- net Net-(U6-EN): vias 3 -> 2
- added copper zone on F.Cu, net GND

Commit message: layout amelioré V67
Parts:
- moved H5 2.67 mm to (125.0, 50.4), turned to 180 degrees
- moved C16 2.19 mm to (157.5, 54.3)
- moved C17 2.19 mm to (157.5, 56.6)
- moved C13 1.55 mm to (121.5, 46.5)
- moved C14 1.10 mm to (177.5, 26.0)
Routing:
- net +5V: track 92.9 -> 101.1 mm
- net +3.6V: track 28.8 -> 32.9 mm, vias 1 -> 2
- net Net-(U4-EN): track 14.4 -> 11.4 mm
- net +3.3V: track 118.9 -> 119.9 mm
- net Net-(U6-EN): track 36.4 -> 35.4 mm
- net /D+: track 55.5 -> 56.5 mm
- net GND: track 176.2 -> 177.1 mm, vias 14 -> 15
- removed copper zone on F.Cu, net GND
