File: _restore_backup_2026-10-02T15-19-04-182/Human_Tracker.kicad_pcb (KiCad board)
At the start: 4 copper layers, 200 x 50 mm, 59 parts, among them U1 TPS54233QDRQ1, U2 ICS-43434_C5656610, U3 ICS-43434_C5656610, U4 ADM7172ACPZ-3.3-R7, U5 BME680, U6 ESP32-S3-WROOM-1(N16R8), U7 MLX90640ESF-BAB-000-TU, U8 FRC0805F1400TS 140

Commit message: commit
Parts:
- moved R3 10.2 mm to (143.7, 68.6), turned to -90 degrees
Routing:
- net GND: track 156.7 -> 333.9 mm, vias 9 -> 8
- net +3.3V: track 113.3 -> 194.9 mm, vias 9 -> 10
- net Net-(USB1-CC1): track 8.23 -> 0.00 mm, vias 2 -> 0
- net +5V: track 92.9 -> 88.3 mm
